File: 02_electronics/kicad/FrostChain_ESkin_Crate.kicad_sch (KiCad schematic)
At the start: 36 parts, among them J1 Fan tach input (verify pinout), Q1 2N7002, U1 MPPT charger, 4S LiFePO4, CV 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, U2 LM2596-5.0, U3 Sipeed Tang Nano 9K (Gowin GW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, U4 ESP32-S3, U5 SIM7600-class 5G/LTE + GNSS m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, U6 12 V -> 4.0 V buck, 3 A, U7 SHT31, U8 BTS7960 module (IBT-2), 43 A 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

Commit message: Add files via upload
Connections:
- net +5V: now also C2.1, L1.2, U2.5 (FB)
